Commit message: Correcting URDF and adding documentation links

File: myworkcell_support/urdf/workcell_gazebo_trial1.urdf (robot description, URDF)
Before this commit: robot myworkcell, 18 links, 17 joints
Links:
- removed link camera_frame
Joints:
- removed joint world_to_camera
- joint camera_depth_joint: origin xyz=0 0.011 0 rpy=0 0 0 -> xyz=0 -0.012 0 rpy=0 0 -1.5707
- joint camera_rgb_joint: origin xyz=0 -0.012 0 rpy=0 0 0 -> xyz=0 -0.012 0 rpy=0 0 -1.5707
- joint wrist_1_joint: limit lower=-3.14159265359 upper=3.14159265359 effort=28.0 velocity=3.2 -> lower=-0.75 upper=0.75 effort=28.0 velocity=3.2
- joint wrist_3_joint: limit lower=-3.14159265359 upper=3.14159265359 effort=28.0 velocity=3.2 -> lower=-0.314 upper=+0.314 effort=28.0 velocity=3.2
